Commit message: Initial commit: LQR ROS2 Gazebo AUV project

File: src/auv_description/urdf/simple_auv.urdf.xacro (robot description, xacro)
@@ -1,4 +1,5 @@
 <?xml version="1.0"?>
-<robot name="simple_auv" xmlns:xacro="http://www.ros.org/wiki/xacro">
+<robot name="simple_auv"
+       xmlns:xacro="http://www.ros.org/wiki/xacro">
   <!-- AUV size and mass parameters -->
   <xacro:property name="auv_length" value="1.0"/>
@@ -7,10 +8,15 @@
   <!-- Main body of the AUV -->
   <link name="base_link">
-    <!-- What the AUV looks like in Gazebo/RViz -->
+    <!-- ============================= -->
+    <!-- Visual model: cylinder -->
+    <!-- ============================= -->
     <visual>
       <!-- Cylinder is along z by default, rotate it to x direction -->
-      <origin xyz="0 0 0" rpy="0 1.57079632679 0"/>
+      <origin xyz="0 0 0"
+              rpy="0 1.57079632679 0"/>
       <geometry>
-        <cylinder radius="${auv_radius}" length="${auv_length}"/>
+        <cylinder
+          radius="${auv_radius}"
+          length="${auv_length}"/>
       </geometry>
       <material name="blue">
@@ -18,14 +24,22 @@
       </material>
     </visual>
-    <!-- Collision shape used by physics engine -->
+    <!-- ============================= -->
+    <!-- Collision model: cylinder -->
+    <!-- ============================= -->
     <collision>
-      <origin xyz="0 0 0" rpy="0 1.57079632679 0"/>
+      <origin xyz="0 0 0"
+              rpy="0 1.57079632679 0"/>
       <geometry>
-        <cylinder radius="${auv_radius}" length="${auv_length}"/>
+        <cylinder
+          radius="${auv_radius}"
+          length="${auv_length}"/>
       </geometry>
     </collision>
+    <!-- ============================= -->
     <!-- Mass and inertia -->
+    <!-- ============================= -->
     <inertial>
-      <origin xyz="0 0 0" rpy="0 0 0"/>
+      <origin xyz="0 0 0"
+              rpy="0 0 0"/>
       <mass value="${auv_mass}"/>
       <!-- Inertia of a cylinder whose main axis is x -->
@@ -34,7 +48,11 @@
         ixy="0.0"
         ixz="0.0"
-        iyy="${(1.0 / 12.0) * auv_mass * (3.0 * auv_radius * auv_radius + auv_length * auv_length)}"
+        iyy="${(1.0 / 12.0) * auv_mass *
+              (3.0 * auv_radius * auv_radius +
+               auv_length * auv_length)}"
         iyz="0.0"
-        izz="${(1.0 / 12.0) * auv_mass * (3.0 * auv_radius * auv_radius + auv_length * auv_length)}"/>
+        izz="${(1.0 / 12.0) * auv_mass *
+              (3.0 * auv_radius * auv_radius +
+               auv_length * auv_length)}"/>
     </inertial>
   </link>
